File: KiCad/breadboard_comp/ALU_1.sch (KiCad schematic (older format))
At the start: 50 parts, among them U12 74LS08, U17 74LS86, U18 74LS283, U19 74LS245, U20 74LS86, U21 74LS02, U22 74LS08, U23 74LS283, U24 74LS86, U25 74LS245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

Commit message: Computer built
Connections:
- net B0: now also U25.9 (A7); no longer U25.18 (B0)
- net B1: now also U25.8 (A6); no longer U25.17 (B1)
- net B10: now also U19.7 (A5); no longer U19.16 (B2)
- net B11: now also U19.6 (A4); no longer U19.15 (B3)
- net B12: now also U19.5 (A3); no longer U19.14 (B4)
- net B13: now also U19.4 (A2); no longer U19.13 (B5)
- net B14: now also U19.3 (A1); no longer U19.12 (B6)
- net B15: now also U19.2 (A0); no longer U19.11 (B7)
- net B2: now also U25.7 (A5); no longer U25.16 (B2)
- net B3: now also U25.6 (A4); no longer U25.15 (B3)
- net B4: now also U25.5 (A3); no longer U25.14 (B4)
- net B5: now also U25.4 (A2); no longer U25.13 (B5)
- net B6: now also U25.3 (A1); no longer U25.12 (B6)
- net B7: now also U25.2 (A0); no longer U25.11 (B7)
- net B8: now also U19.9 (A7); no longer U19.18 (B0)
- net B9: now also U19.8 (A6); no longer U19.17 (B1)
- net GND: now also U19.1 (A->B), U25.1 (A->B)
- net PF: now also U25.11 (B7); no longer U25.2 (A0)
- net VCC: no longer U19.1 (A->B), U25.1 (A->B)
- net at D41.2 (A), U21.2, U23.4 (S1): now also U19.11 (B7); no longer U19.2 (A0)
- net at D40.2 (A), U21.3, U23.1 (S2): now also U19.12 (B6); no longer U19.3 (A1)
- net at D39.2 (A), U21.5, U23.13 (S3): now also U19.13 (B5); no longer U19.4 (A2)
- net at D38.2 (A), U21.6, U23.10 (S4): now also U19.14 (B4); no longer U19.5 (A3)
- net at D37.2 (A), U18.4 (S1), U21.8: now also U19.15 (B3); no longer U19.6 (A4)
- net at D36.2 (A), U18.1 (S2), U21.9: now also U19.16 (B2); no longer U19.7 (A5)
- net at D35.2 (A), U18.13 (S3), U21.11: now also U19.17 (B1); no longer U19.8 (A6)
- net at D34.2 (A), U18.10 (S4), U21.12: now also U19.18 (B0); no longer U19.9 (A7)
- net at D47.2 (A), U26.3, U30.1 (S2): now also U25.12 (B6); no longer U25.3 (A1)
- net at D48.2 (A), U26.5, U30.13 (S3): now also U25.13 (B5); no longer U25.4 (A2)
- net at D49.2 (A), U26.6, U30.10 (S4): now also U25.14 (B4); no longer U25.5 (A3)
- net at D42.2 (A), U26.8, U27.4 (S1): now also U25.15 (B3); no longer U25.6 (A4)
- net at D43.2 (A), U26.9, U27.1 (S2): now also U25.16 (B2); no longer U25.7 (A5)
- net at D44.2 (A), U26.11, U27.13 (S3): now also U25.17 (B1); no longer U25.8 (A6)
- net at D45.2 (A), U26.12, U27.10 (S4): now also U25.18 (B0); no longer U25.9 (A7)
Other:
- moved on the sheet: D34, D35, D36, D37, R41, R42, R43, R44, U19, U21A, U21B, U21C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
