File: KiCad/breadboard_comp/ALU_1.sch (KiCad schematic (older format))
At the start: 50 parts, among them U12 74LS08, U17 74LS86, U18 74LS283, U19 74LS245, U20 74LS86, U21 74LS02, U22 74LS08, U23 74LS283, U24 74LS86, U25 74LS245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

Commit message: Schematic + Report Progress
Parts:
- added U87: 74LS08, symbol 74xx:74LS08
Connections:
- net SU: now also U87.12, U87.13; no longer U17.1, U17.12, U17.4, U17.9, U20.1, U20.12, U20.4, U20.9
- new net: U17.1, U17.12, U17.4, U17.9, U20.1, U20.12, U20.4, U20.9, U87.11
Changed lines of the file:
@@
 $Descr A3 16535 11693
 encoding utf-8
-Sheet 5 19
+Sheet 5 18
 Title ""
 Date ""
@@
 Wire Wire Line
 	6800 1800 6800 3800
-Text HLabel 10550 650  2    50   Input ~ 0
+Text HLabel 11200 1850 3    50   Input ~ 0
 SU
-Wire Wire Line
-	10550 650  9900 650
 Wire Wire Line
 	9900 650  9900 4500
@@
 Connection ~ 6200 650
 Wire Wire Line
-	5800 650  4800 650
-Connection ~ 5800 650
-Wire Wire Line
 	4800 650  4800 3800
 Wire Wire Line
@@
 Wire Wire Line
 	4400 650  4800 650
-Connection ~ 4800 650
 Wire Wire Line
 	4400 650  4000 650
@@
 Connection ~ 6400 7450
 Connection ~ 6900 6350
+$Comp
+L 74xx:74LS08 U87
+U 4 1 5F47772C
+P 11500 1150
+F 0 "U87" H 11500 950 50  0000 C CNN
+F 1 "74LS08" H 11500 1150 50  0000 C CNN
+F 2 "" H 11500 1150 50  0001 C CNN
+F 3 "http://www.ti.com/lit/gpn/sn74LS08" H 11500 1150 50  0001 C CNN
+	4    11500 1150
+	0    -1   -1   0
+$EndComp
+Wire Wire Line
+	11200 1850 11200 1700
+Wire Wire Line
+	11200 1700 11400 1700
+Wire Wire Line
+	11600 1700 11600 1450
+Wire Wire Line
+	11400 1450 11400 1700
+Connection ~ 11400 1700
+Wire Wire Line
+	11400 1700 11600 1700
+Wire Wire Line
+	11200 1700 11200 650
+Wire Wire Line
+	9900 650  11200 650
+Connection ~ 11200 1700
+Wire Wire Line
+	4800 650  4950 650
+Wire Wire Line
+	4950 650  4950 550
+Wire Wire Line
+	4950 550  11500 550
+Wire Wire Line
+	11500 550  11500 850
 Wire Bus Line
 	1650 10600 6400 10600
+Connection ~ 4800 650
 $EndSCHEMATC
