File: KiCad/breadboard_comp/A_register.sch (KiCad schematic (older format))
At the start: 38 parts, among them U10 74LS245, U11 74LS245, U7 74LS08, U8 74LS273, U9 74LS273

Commit message: Computer built
Connections:
- net A0: now also U11.11 (B7); no longer U11.18 (B0)
- net A1: now also U11.12 (B6); no longer U11.17 (B1)
- net A10: now also U10.13 (B5); no longer U10.16 (B2)
- net A11: now also U10.14 (B4); no longer U10.15 (B3)
- net A12: now also U10.15 (B3); no longer U10.14 (B4)
- net A13: now also U10.16 (B2); no longer U10.13 (B5)
- net A14: now also U10.17 (B1); no longer U10.12 (B6)
- net A15: now also U10.18 (B0); no longer U10.11 (B7)
- net A2: now also U11.13 (B5); no longer U11.16 (B2)
- net A3: now also U11.14 (B4); no longer U11.15 (B3)
- net A4: now also U11.15 (B3); no longer U11.14 (B4)
- net A5: now also U11.16 (B2); no longer U11.13 (B5)
- net A6: now also U11.17 (B1); no longer U11.12 (B6)
- net A7: now also U11.18 (B0); no longer U11.11 (B7)
- net A8: now also U10.11 (B7); no longer U10.18 (B0)
- net A9: now also U10.12 (B6); no longer U10.17 (B1)
- net B0: now also U11.9 (A7); no longer U11.2 (A0)
- net B1: now also U11.8 (A6); no longer U11.3 (A1)
- net B10: now also U10.7 (A5); no longer U10.4 (A2)
- net B11: now also U10.6 (A4); no longer U10.5 (A3)
- net B12: now also U10.5 (A3); no longer U10.6 (A4)
- net B13: now also U10.4 (A2); no longer U10.7 (A5)
- net B14: now also U10.3 (A1); no longer U10.8 (A6)
- net B15: now also U10.2 (A0); no longer U10.9 (A7)
- net B2: now also U11.7 (A5); no longer U11.4 (A2)
- net B3: now also U11.6 (A4); no longer U11.5 (A3)
- net B4: now also U11.5 (A3); no longer U11.6 (A4)
- net B5: now also U11.4 (A2); no longer U11.7 (A5)
- net B6: now also U11.3 (A1); no longer U11.8 (A6)
- net B7: now also U11.2 (A0); no longer U11.9 (A7)
- net B8: now also U10.9 (A7); no longer U10.2 (A0)
- net B9: now also U10.8 (A6); no longer U10.3 (A1)
