File: KiCad/breadboard_comp/C_register.sch (KiCad schematic (older format))
At the start: 38 parts, among them U38 74LS08, U39 74LS273, U40 74LS273, U41 74LS245, U42 74LS245

Commit message: Computer built
Connections:
- net B0: now also U42.9 (A7); no longer U42.2 (A0)
- net B1: now also U42.8 (A6); no longer U42.3 (A1)
- net B10: now also U41.7 (A5); no longer U41.4 (A2)
- net B11: now also U41.6 (A4); no longer U41.5 (A3)
- net B12: now also U41.5 (A3); no longer U41.6 (A4)
- net B13: now also U41.4 (A2); no longer U41.7 (A5)
- net B14: now also U41.3 (A1); no longer U41.8 (A6)
- net B15: now also U41.2 (A0); no longer U41.9 (A7)
- net B2: now also U42.7 (A5); no longer U42.4 (A2)
- net B3: now also U42.6 (A4); no longer U42.5 (A3)
- net B4: now also U42.5 (A3); no longer U42.6 (A4)
- net B5: now also U42.4 (A2); no longer U42.7 (A5)
- net B6: now also U42.3 (A1); no longer U42.8 (A6)
- net B7: now also U42.2 (A0); no longer U42.9 (A7)
- net B8: now also U41.9 (A7); no longer U41.2 (A0)
- net B9: now also U41.8 (A6); no longer U41.3 (A1)
- net at D62.2 (A), U40.9 (Q3): now also U42.14 (B4); no longer U42.15 (B3)
- net at D63.2 (A), U40.6 (Q2): now also U42.13 (B5); no longer U42.16 (B2)
- net at D58.2 (A), U40.19 (Q7): now also U42.18 (B0); no longer U42.11 (B7)
- net at D50.2 (A), U39.19 (Q7): now also U41.18 (B0); no longer U41.11 (B7)
- net at D64.2 (A), U40.5 (Q1): now also U42.12 (B6); no longer U42.17 (B1)
- net at D52.2 (A), U39.15 (Q5): now also U41.16 (B2); no longer U41.13 (B5)
- net at D53.2 (A), U39.12 (Q4): now also U41.15 (B3); no longer U41.14 (B4)
- net at D55.2 (A), U39.6 (Q2): now also U41.13 (B5); no longer U41.16 (B2)
- net at D60.2 (A), U40.15 (Q5): now also U42.16 (B2); no longer U42.13 (B5)
- net at D51.2 (A), U39.16 (Q6): now also U41.17 (B1); no longer U41.12 (B6)
- net at D57.2 (A), U39.2 (Q0): now also U41.11 (B7); no longer U41.18 (B0)
- net at D56.2 (A), U39.5 (Q1): now also U41.12 (B6); no longer U41.17 (B1)
- net at D54.2 (A), U39.9 (Q3): now also U41.14 (B4); no longer U41.15 (B3)
- net at D61.2 (A), U40.12 (Q4): now also U42.15 (B3); no longer U42.14 (B4)
- net at D59.2 (A), U40.16 (Q6): now also U42.17 (B1); no longer U42.12 (B6)
- net at D65.2 (A), U40.2 (Q0): now also U42.11 (B7); no longer U42.18 (B0)
Changed lines of the file:
@@
 Wire Wire Line
 	9500 2500 9500 3250
-Text Label 9500 2600 1    50   ~ 0
+Text Label 8800 2600 1    50   ~ 0
 B0
-Text Label 9400 2650 1    50   ~ 0
+Text Label 8900 2650 1    50   ~ 0
 B1
-Text Label 9300 2750 1    50   ~ 0
+Text Label 9000 2750 1    50   ~ 0
 B2
-Text Label 9200 2800 1    50   ~ 0
+Text Label 9100 2800 1    50   ~ 0
 B3
-Text Label 9100 2850 1    50   ~ 0
+Text Label 9200 2850 1    50   ~ 0
 B4
-Text Label 9000 2900 1    50   ~ 0
+Text Label 9300 2900 1    50   ~ 0
 B5
-Text Label 8900 2950 1    50   ~ 0
+Text Label 9400 2950 1    50   ~ 0
 B6
-Text Label 8800 3000 1    50   ~ 0
+Text Label 9500 3000 1    50   ~ 0
 B7
 Entry Wire Line
@@
 Wire Wire Line
 	7350 2500 7350 3250
-Text Label 7350 2600 1    50   ~ 0
+Text Label 6650 2600 1    50   ~ 0
 B8
-Text Label 7250 2650 1    50   ~ 0
+Text Label 6750 2650 1    50   ~ 0
 B9
-Text Label 7150 2750 1    50   ~ 0
+Text Label 6850 2750 1    50   ~ 0
 B10
-Text Label 7050 2800 1    50   ~ 0
+Text Label 6950 2800 1    50   ~ 0
 B11
-Text Label 6950 2850 1    50   ~ 0
+Text Label 7050 2850 1    50   ~ 0
 B12
-Text Label 6850 2900 1    50   ~ 0
+Text Label 7150 2900 1    50   ~ 0
 B13
-Text Label 6750 2950 1    50   ~ 0
+Text Label 7250 2950 1    50   ~ 0
 B14
-Text Label 6650 3000 1    50   ~ 0
+Text Label 7350 3000 1    50   ~ 0
 B15
 Wire Wire Line
 	2650 4250 2650 4650
 Wire Wire Line
-	7350 4650 7350 4250
-Wire Wire Line
 	2550 4250 2550 4750
 Wire Wire Line
-	7250 4750 7250 4250
-Wire Wire Line
 	2450 4250 2450 4850
 Wire Wire Line
-	7150 4850 7150 4250
-Wire Wire Line
 	2350 4250 2350 4950
 Wire Wire Line
-	7050 4950 7050 4250
-Wire Wire Line
 	2250 4250 2250 5050
 Wire Wire Line
 	2250 5050 3550 5050
 Wire Wire Line
-	6950 5050 6950 4250
-Wire Wire Line
 	2150 4250 2150 5150
 Wire Wire Line
 	2150 5150 3350 5150
 Wire Wire Line
-	6850 5150 6850 4250
-Wire Wire Line
 	2050 4250 2050 5250
 Wire Wire Line
 	2050 5250 3150 5250
 Wire Wire Line
-	6750 5250 6750 4250
-Wire Wire Line
 	1950 4250 1950 5350
 Wire Wire Line
 	1950 5350 2950 5350
 Wire Wire Line
-	6650 5350 6650 4250
-Wire Wire Line
 	5150 4250 5150 5650
 Wire Wire Line
-	9500 5650 9500 4250
-Wire Wire Line
 	5050 4250 5050 5750
 Wire Wire Line
-	9400 5750 9400 4250
-Wire Wire Line
 	4950 4250 4950 5850
 Wire Wire Line
 	4950 5850 5550 5850
 Wire Wire Line
-	9300 5850 9300 4250
-Wire Wire Line
 	4850 4250 4850 5950
 Wire Wire Line
-	9200 5950 9200 4250
-Wire Wire Line
 	4750 4250 4750 6050
 Wire Wire Line
-	9100 6050 9100 4250
-Wire Wire Line
 	4650 4250 4650 6150
 Wire Wire Line
-	9000 6150 9000 4250
-Wire Wire Line
 	4550 4250 4550 6250
 Wire Wire Line
-	8900 6250 8900 4250
-Wire Wire Line
 	4450 4250 4450 6350
 Wire Wire Line
 	4450 6350 4550 6350
-Wire Wire Line
-	8800 6350 8800 4250
 $Comp
 L power:GND #PWR?
@@
 Connection ~ 4350 4650
 Wire Wire Line
-	4350 4650 7350 4650
+	4350 4650 6650 4650
 Wire Wire Line
 	4150 4750 4150 6700
 Connection ~ 4150 4750
 Wire Wire Line
-	4150 4750 7250 4750
+	4150 4750 6750 4750
 Wire Wire Line
 	3950 6700 3950 4850
 Connection ~ 3950 4850
 Wire Wire Line
-	3950 4850 7150 4850
+	3950 4850 6850 4850
 Wire Wire Line
 	3750 4950 3750 6700
 Connection ~ 3750 4950
 Wire Wire Line
-	3750 4950 7050 4950
+	3750 4950 6950 4950
 Wire Wire Line
 	3550 5050 3550 6700
 Connection ~ 3550 5050
 Wire Wire Line
-	3550 5050 6950 5050
-Wire Wire Line
 	3350 5150 3350 6700
 Connection ~ 3350 5150
 Wire Wire Line
-	3350 5150 6850 5150
-Wire Wire Line
 	3150 6700 3150 5250
 Connection ~ 3150 5250
 Wire Wire Line
-	3150 5250 6750 5250
-Wire Wire Line
 	2950 5350 2950 6700
 Connection ~ 2950 5350
 Wire Wire Line
-	2950 5350 6650 5350
-Wire Wire Line
 	4550 6700 4550 6350
 Connection ~ 4550 6350
 Wire Wire Line
-	4550 6350 8800 6350
-Wire Wire Line
 	4750 6700 4750 6250
 Wire Wire Line
@@
 Connection ~ 4750 6250
 Wire Wire Line
-	4750 6250 8900 6250
-Wire Wire Line
 	4950 6700 4950 6150
 Wire Wire Line
@@
 Connection ~ 4950 6150
 Wire Wire Line
-	4950 6150 9000 6150
-Wire Wire Line
 	5150 6700 5150 6050
 Wire Wire Line
@@
 Connection ~ 5150 6050
 Wire Wire Line
-	5150 6050 9100 6050
-Wire Wire Line
 	5350 6700 5350 5950
 Wire Wire Line
@@
 Connection ~ 5350 5950
 Wire Wire Line
-	5350 5950 9200 5950
+	5350 5950 9100 5950
 Wire Wire Line
 	5550 6700 5550 5850
 Connection ~ 5550 5850
 Wire Wire Line
-	5550 5850 9300 5850
+	5550 5850 9000 5850
 Wire Wire Line
 	5750 6700 5750 5750
@@
 Connection ~ 5750 5750
 Wire Wire Line
-	5750 5750 9400 5750
+	5750 5750 8900 5750
 Wire Wire Line
 	5950 6700 5950 5650
@@
 Connection ~ 5950 5650
 Wire Wire Line
-	5950 5650 9500 5650
+	5950 5650 8800 5650
 Wire Wire Line
 	1250 2150 6350 2150
@@
 Wire Wire Line
 	750  1800 1000 1800
+Text HLabel 9600 2400 2    50   BiDi ~ 0
+BUS
+Wire Wire Line
+	8800 4250 8800 5650
+Wire Wire Line
+	8900 5750 8900 4250
+Wire Wire Line
+	9000 4250 9000 5850
+Wire Wire Line
+	9100 5950 9100 4250
+Wire Wire Line
+	5150 6050 9200 6050
+Wire Wire Line
+	9200 4250 9200 6050
+Wire Wire Line
+	9300 6150 9300 4250
+Wire Wire Line
+	4950 6150 9300 6150
+Wire Wire Line
+	9400 4250 9400 6250
+Wire Wire Line
+	4750 6250 9400 6250
+Wire Wire Line
+	9500 6350 9500 4250
+Wire Wire Line
+	4550 6350 9500 6350
+Wire Wire Line
+	6650 4250 6650 4650
+Wire Wire Line
+	6750 4750 6750 4250
+Wire Wire Line
+	6850 4250 6850 4850
+Wire Wire Line
+	6950 4950 6950 4250
+Wire Wire Line
+	3550 5050 7050 5050
+Wire Wire Line
+	7050 4250 7050 5050
+Wire Wire Line
+	7150 5150 7150 4250
+Wire Wire Line
+	3350 5150 7150 5150
+Wire Wire Line
+	7250 4250 7250 5250
+Wire Wire Line
+	3150 5250 7250 5250
+Wire Wire Line
+	7350 5350 7350 4250
+Wire Wire Line
+	2950 5350 7350 5350
 Wire Bus Line
 	1850 2400 9600 2400
-Text HLabel 9600 2400 2    50   BiDi ~ 0
-BUS
 $EndSCHEMATC
