File: KiCad/breadboard_comp/Display.sch (KiCad schematic (older format))
At the start: 6 parts, among them U66 74LS00, U67 74LS245, U68 74LS245, U69 MC21605C6W

Commit message: Computer built
Parts:
- removed U66: 74LS00, symbol 74xx:74LS00
- added U105: 74LS08, symbol 74xx:74LS08
- added U66: 74LS04, symbol 74xx:74LS04
- R103: value R_Variable -> 20k
Connections:
- net B10 is gone; now on net GND: U67.7 (A5)
- net B9 is gone; now on net GND: U67.8 (A6)
- net CLK: now also U105.1
- net GND: now also U67.12 (B6), U67.13 (B5), U69.5 (R/~W)
- net OUT: now also U105.2, U66.1
- net at U69.6 (E): now also U105.3; no longer U67.13 (B5)
- net at U67.19 (CE), U68.19 (CE): now also U66.2
Changed lines of the file:
@@
 $Descr A4 11693 8268
 encoding utf-8
-Sheet 13 18
+Sheet 12 18
 Title ""
 Date ""
@@
 P 6000 4100
 F 0 "R103" H 6128 4146 50  0000 L CNN
-F 1 "R_Variable" H 6128 4055 50  0000 L CNN
+F 1 "20k" H 6128 4055 50  0000 L CNN
 F 2 "" V 5930 4100 50  0001 C CNN
 F 3 "~" H 6000 4100 50  0001 C CNN
@@
 Wire Wire Line
 	4650 2600 4150 2600
-Wire Wire Line
-	4150 2500 4750 2500
-Wire Wire Line
-	4750 2500 4750 3700
-Wire Wire Line
-	4750 3700 5150 3700
-Wire Wire Line
-	5150 3600 4850 3600
-Wire Wire Line
-	4850 3600 4850 2400
-Wire Wire Line
-	4850 2400 4150 2400
-$Comp
-L power:GND #PWR0167
-U 1 1 5F491E9C
-P 4750 2100
-F 0 "#PWR0167" H 4750 1850 50  0001 C CNN
-F 1 "GND" V 4755 1972 50  0000 R CNN
-F 2 "" H 4750 2100 50  0001 C CNN
-F 3 "" H 4750 2100 50  0001 C CNN
-	1    4750 2100
-	0    -1   -1   0
-$EndComp
-Wire Wire Line
-	4750 2100 4650 2100
-Wire Wire Line
-	4150 2000 4650 2000
-Wire Wire Line
-	4650 2000 4650 2100
-Connection ~ 4650 2100
-Wire Wire Line
-	4650 2100 4150 2100
-Wire Wire Line
-	4650 2000 4650 1900
-Wire Wire Line
-	4650 1900 4150 1900
-Connection ~ 4650 2000
-Wire Wire Line
-	4150 2300 4650 2300
-Wire Wire Line
-	4650 2300 4650 2200
-Wire Wire Line
-	4650 2200 4150 2200
-Connection ~ 4650 2200
-Wire Wire Line
-	4650 2200 4650 2100
-Entry Wire Line
-	1950 2400 2050 2500
 Entry Wire Line
 	1950 2500 2050 2600
@@
 Entry Wire Line
 	1950 4500 2050 4600
-Entry Wire Line
-	1950 2300 2050 2400
-Wire Wire Line
-	2050 2400 3150 2400
-Wire Wire Line
-	3150 2500 2050 2500
 Wire Wire Line
 	2050 2600 3150 2600
-$Comp
-L power:GND #PWR0160
-U 1 1 5F49AAE3
-P 2500 2100
-F 0 "#PWR0160" H 2500 1850 50  0001 C CNN
-F 1 "GND" V 2505 1972 50  0000 R CNN
-F 2 "" H 2500 2100 50  0001 C CNN
-F 3 "" H 2500 2100 50  0001 C CNN
-	1    2500 2100
-	0    1    1    0
-$EndComp
-Wire Wire Line
-	2500 2100 2650 2100
-Wire Wire Line
-	3150 2000 2650 2000
-Wire Wire Line
-	2650 2000 2650 2100
-Connection ~ 2650 2100
-Wire Wire Line
-	2650 2100 3150 2100
-Wire Wire Line
-	2650 2100 2650 2200
-Wire Wire Line
-	2650 2200 3150 2200
-Wire Wire Line
-	3150 2300 2650 2300
-Wire Wire Line
-	2650 2300 2650 2200
-Connection ~ 2650 2200
-Wire Wire Line
-	2650 2000 2650 1900
-Wire Wire Line
-	2650 1900 3150 1900
-Connection ~ 2650 2000
 $Comp
 L power:VCC #PWR0165
@@
 L power:GND #PWR0163
 U 1 1 5F4A231B
-P 3500 3350
-F 0 "#PWR0163" H 3500 3100 50  0001 C CNN
-F 1 "GND" V 3505 3222 50  0000 R CNN
-F 2 "" H 3500 3350 50  0001 C CNN
-F 3 "" H 3500 3350 50  0001 C CNN
-	1    3500 3350
-	0    1    1    0
-$EndComp
-Wire Wire Line
-	3500 3350 3650 3350
-Wire Wire Line
-	3650 3350 3650 3200
+P 3500 3250
+F 0 "#PWR0163" H 3500 3000 50  0001 C CNN
+F 1 "GND" V 3505 3122 50  0000 R CNN
+F 2 "" H 3500 3250 50  0001 C CNN
+F 3 "" H 3500 3250 50  0001 C CNN
+	1    3500 3250
+	0    1    1    0
+$EndComp
+Wire Wire Line
+	3500 3250 3650 3250
 $Comp
 L power:VCC #PWR0166
@@
 Wire Wire Line
 	3000 2800 3150 2800
-Wire Wire Line
-	2400 5550 2400 4900
-Wire Wire Line
-	2400 2900 3150 2900
-Wire Wire Line
-	3150 4900 2400 4900
-Connection ~ 2400 4900
-Wire Wire Line
-	2400 4900 2400 2900
 Text Notes 1900 3700 1    50   ~ 10
 16-Bit Common Bus
-Text Label 2150 4600 0    50   ~ 0
-B0
-Text Label 2150 4500 0    50   ~ 0
-B1
-Text Label 2150 4400 0    50   ~ 0
-B2
-Text Label 2150 4300 0    50   ~ 0
-B3
-Text Label 2150 4200 0    50   ~ 0
-B4
-Text Label 2150 4100 0    50   ~ 0
-B5
-Text Label 2150 4000 0    50   ~ 0
-B6
-Text Label 2150 3900 0    50   ~ 0
-B7
 Text Label 2150 2600 0    50   ~ 0
 B8
-Text Label 2150 2500 0    50   ~ 0
-B9
-Text Label 2150 2400 0    50   ~ 0
-B10
 $Comp
 L power:VCC #PWR?
@@
 Wire Wire Line
 	5950 2050 5950 2150
-Text HLabel 2300 6250 3    50   Input ~ 0
+Text HLabel 2400 6150 3    50   Input ~ 0
 OUT
-Text HLabel 2500 6250 3    50   Input ~ 0
+Text HLabel 2350 3300 0    50   Input ~ 0
 CLK
-$Comp
-L 74xx:74LS00 U66
-U 1 1 5F4EE5EB
-P 2400 5850
-F 0 "U66" V 2446 5670 50  0000 R CNN
-F 1 "74LS00" V 2400 6000 50  0000 R CNN
-F 2 "" H 2400 5850 50  0001 C CNN
-F 3 "http://www.ti.com/lit/gpn/sn74ls00" H 2400 5850 50  0001 C CNN
-	1    2400 5850
-	0    -1   -1   0
-$EndComp
-Wire Wire Line
-	2300 6250 2300 6150
-Wire Wire Line
-	2500 6250 2500 6150
 Text HLabel 1950 4900 3    50   BiDi ~ 0
 BUS
+Connection ~ 4650 2200
+Wire Wire Line
+	4650 2200 4150 2200
+Wire Wire Line
+	4650 2300 4650 2200
+Wire Wire Line
+	4150 2300 4650 2300
+Connection ~ 4650 2000
+Wire Wire Line
+	4650 1900 4150 1900
+Wire Wire Line
+	4650 2000 4650 1900
+Wire Wire Line
+	4650 2100 4150 2100
+Connection ~ 4650 2100
+Wire Wire Line
+	4650 2000 4650 2100
+Wire Wire Line
+	4150 2000 4650 2000
+Wire Wire Line
+	4750 2200 4650 2200
+$Comp
+L power:GND #PWR0167
+U 1 1 5F491E9C
+P 4750 2200
+F 0 "#PWR0167" H 4750 1950 50  0001 C CNN
+F 1 "GND" V 4755 2072 50  0000 R CNN
+F 2 "" H 4750 2200 50  0001 C CNN
+F 3 "" H 4750 2200 50  0001 C CNN
+	1    4750 2200
+	0    -1   -1   0
+$EndComp
+Connection ~ 2650 2000
+Wire Wire Line
+	2650 1900 3150 1900
+Wire Wire Line
+	2650 2000 2650 1900
+Connection ~ 2650 2200
+Wire Wire Line
+	2650 2300 2650 2200
+Wire Wire Line
+	3150 2300 2650 2300
+Wire Wire Line
+	2650 2200 3150 2200
+Wire Wire Line
+	2650 2100 3150 2100
+Connection ~ 2650 2100
+Wire Wire Line
+	2650 2000 2650 2100
+Wire Wire Line
+	3150 2000 2650 2000
+$Comp
+L power:GND #PWR0160
+U 1 1 5F49AAE3
+P 2500 2200
+F 0 "#PWR0160" H 2500 1950 50  0001 C CNN
+F 1 "GND" V 2505 2072 50  0000 R CNN
+F 2 "" H 2500 2200 50  0001 C CNN
+F 3 "" H 2500 2200 50  0001 C CNN
+	1    2500 2200
+	0    1    1    0
+$EndComp
+Text Label 2150 4200 0    50   ~ 0
+B4
+Text Label 2150 4300 0    50   ~ 0
+B3
+Text Label 2150 4100 0    50   ~ 0
+B5
+Text Label 2150 4400 0    50   ~ 0
+B2
+Text Label 2150 4000 0    50   ~ 0
+B6
+Text Label 2150 4500 0    50   ~ 0
+B1
+Text Label 2150 4600 0    50   ~ 0
+B0
+Text Label 2150 3900 0    50   ~ 0
+B7
+Wire Wire Line
+	3150 2400 2650 2400
+Wire Wire Line
+	2650 2400 2650 2300
+Connection ~ 2650 2300
+Wire Wire Line
+	2500 2200 2650 2200
+Wire Wire Line
+	4150 2400 4650 2400
+Wire Wire Line
+	4650 2400 4650 2300
+Connection ~ 4650 2300
+$Comp
+L 74xx:74LS08 U105
+U 1 1 5EB9CB63
+P 2850 3400
+F 0 "U105" H 2800 3600 50  0000 C CNN
+F 1 "74LS08" H 2850 3400 50  0000 C CNN
+F 2 "" H 2850 3400 50  0001 C CNN
+F 3 "http://www.ti.com/lit/gpn/sn74LS08" H 2850 3400 50  0001 C CNN
+	1    2850 3400
+	1    0    0    -1
+$EndComp
+Wire Wire Line
+	3650 3250 3650 3200
+Wire Wire Line
+	2350 3300 2550 3300
+Wire Wire Line
+	2550 3500 2400 3500
+$Comp
+L 74xx:74LS04 U66
+U 1 1 5EBAA100
+P 2600 5300
+F 0 "U66" V 2750 5200 50  0000 R CNN
+F 1 "74LS04" V 2500 5450 50  0000 R CNN
+F 2 "" H 2600 5300 50  0001 C CNN
+F 3 "http://www.ti.com/lit/gpn/sn74LS04" H 2600 5300 50  0001 C CNN
+	1    2600 5300
+	0    -1   -1   0
+$EndComp
+Wire Wire Line
+	2400 5800 2600 5800
+Wire Wire Line
+	2600 5800 2600 5600
+Connection ~ 2400 5800
+Wire Wire Line
+	2400 5800 2400 6150
+Wire Wire Line
+	2400 3500 2400 5800
+Wire Wire Line
+	2600 5000 2600 4900
+Wire Wire Line
+	2600 4900 3150 4900
+Wire Wire Line
+	2600 4900 2600 3650
+Wire Wire Line
+	2600 3650 2050 3650
+Wire Wire Line
+	2050 3650 2050 2900
+Connection ~ 2600 4900
+Wire Wire Line
+	2050 2900 3150 2900
+Wire Wire Line
+	3150 3400 5000 3400
+Wire Wire Line
+	5000 3400 5000 3600
+Wire Wire Line
+	5000 3600 5150 3600
+$Comp
+L power:GND #PWR0140
+U 1 1 5EBBD185
+P 5000 3700
+F 0 "#PWR0140" H 5000 3450 50  0001 C CNN
+F 1 "GND" V 5005 3572 50  0000 R CNN
+F 2 "" H 5000 3700 50  0001 C CNN
+F 3 "" H 5000 3700 50  0001 C CNN
+	1    5000 3700
+	0    1    1    0
+$EndComp
+Wire Wire Line
+	5000 3700 5150 3700
+Wire Wire Line
+	3150 2500 2650 2500
+Wire Wire Line
+	2650 2500 2650 2400
+Connection ~ 2650 2400
+Wire Wire Line
+	4650 2400 4650 2500
+Wire Wire Line
+	4650 2500 4150 2500
+Connection ~ 4650 2400
+Wire Wire Line
+	2650 2100 2650 2200
+Wire Wire Line
+	4650 2100 4650 2200
 Wire Bus Line
 	1950 1700 1950 4900
