File: KiCad/breadboard_comp/Display.sch (KiCad schematic (older format))
At the start: 7 parts, among them U105 74LS08, U66 74LS04, U67 74LS245, U68 74LS245, U69 MC21605C6W

Commit message: Schematic + Report Progress
Parts:
- removed U105: 74LS08, symbol 74xx:74LS08
- removed U66: 74LS04, symbol 74xx:74LS04
Connections:
- net GND: now also U67.19 (CE), U68.19 (CE)
- net OUT: now also U69.6 (E)
Changed lines of the file:
@@
 $Descr A4 11693 8268
 encoding utf-8
-Sheet 12 19
+Sheet 12 18
 Title ""
 Date ""
@@
 Wire Wire Line
 	5950 2050 5950 2150
-Text HLabel 2400 6150 3    50   Input ~ 0
+Text HLabel 5000 3600 0    50   Input ~ 0
 OUT
-Text HLabel 2350 3300 0    50   Input ~ 0
-CLK
 Text HLabel 1950 4900 3    50   BiDi ~ 0
 BUS
@@
 	4650 2400 4650 2300
 Connection ~ 4650 2300
-$Comp
-L 74xx:74LS08 U105
-U 1 1 5EB9CB63
-P 2850 3400
-F 0 "U105" H 2800 3600 50  0000 C CNN
-F 1 "74LS08" H 2850 3400 50  0000 C CNN
-F 2 "" H 2850 3400 50  0001 C CNN
-F 3 "http://www.ti.com/lit/gpn/sn74LS08" H 2850 3400 50  0001 C CNN
-	1    2850 3400
-	1    0    0    -1
-$EndComp
 Wire Wire Line
 	3650 3250 3650 3200
-Wire Wire Line
-	2350 3300 2550 3300
-Wire Wire Line
-	2550 3500 2400 3500
-$Comp
-L 74xx:74LS04 U66
-U 1 1 5EBAA100
-P 2600 5300
-F 0 "U66" V 2750 5200 50  0000 R CNN
-F 1 "74LS04" V 2500 5450 50  0000 R CNN
-F 2 "" H 2600 5300 50  0001 C CNN
-F 3 "http://www.ti.com/lit/gpn/sn74LS04" H 2600 5300 50  0001 C CNN
-	1    2600 5300
-	0    -1   -1   0
-$EndComp
-Wire Wire Line
-	2400 5800 2600 5800
-Wire Wire Line
-	2600 5800 2600 5600
-Connection ~ 2400 5800
-Wire Wire Line
-	2400 5800 2400 6150
-Wire Wire Line
-	2400 3500 2400 5800
-Wire Wire Line
-	2600 5000 2600 4900
-Wire Wire Line
-	2600 4900 3150 4900
-Wire Wire Line
-	2600 4900 2600 3650
-Wire Wire Line
-	2600 3650 2050 3650
-Wire Wire Line
-	2050 3650 2050 2900
-Connection ~ 2600 4900
-Wire Wire Line
-	2050 2900 3150 2900
-Wire Wire Line
-	3150 3400 5000 3400
-Wire Wire Line
-	5000 3400 5000 3600
 Wire Wire Line
 	5000 3600 5150 3600
@@
 Wire Wire Line
 	4650 2100 4650 2200
+Wire Wire Line
+	3150 4900 3150 5200
+Wire Wire Line
+	3150 5200 3650 5200
+Connection ~ 3650 5200
+Wire Wire Line
+	3150 3200 3650 3200
+Wire Wire Line
+	3150 2900 3150 3200
 Wire Bus Line
 	1950 1700 1950 4900
+Connection ~ 3650 3200
 $EndSCHEMATC
