File: KiCad/breadboard_comp/Input_Output.sch (KiCad schematic (older format))
At the start: 3 parts, among them U70 74LS245, U71 74LS245

Commit message: Computer built
Connections:
- net ARDUINO_IO_0: now also U71.11 (B7); no longer U70.11 (B7)
- net ARDUINO_IO_1: now also U71.12 (B6); no longer U70.12 (B6)
- net ARDUINO_IO_10: now also U70.13 (B5); no longer U71.13 (B5)
- net ARDUINO_IO_11: now also U70.14 (B4); no longer U71.14 (B4)
- net ARDUINO_IO_12: now also U70.15 (B3); no longer U71.15 (B3)
- net ARDUINO_IO_13: now also U70.16 (B2); no longer U71.16 (B2)
- net ARDUINO_IO_14: now also U70.17 (B1); no longer U71.17 (B1)
- net ARDUINO_IO_15: now also U70.18 (B0); no longer U71.18 (B0)
- net ARDUINO_IO_2: now also U71.13 (B5); no longer U70.13 (B5)
- net ARDUINO_IO_3: now also U71.14 (B4); no longer U70.14 (B4)
- net ARDUINO_IO_4: now also U71.15 (B3); no longer U70.15 (B3)
- net ARDUINO_IO_5: now also U71.16 (B2); no longer U70.16 (B2)
- net ARDUINO_IO_6: now also U71.17 (B1); no longer U70.17 (B1)
- net ARDUINO_IO_7: now also U71.18 (B0); no longer U70.18 (B0)
- net ARDUINO_IO_8: now also U70.11 (B7); no longer U71.11 (B7)
- net ARDUINO_IO_9: now also U70.12 (B6); no longer U71.12 (B6)
- net B0: now also U71.9 (A7); no longer U71.2 (A0)
- net B1: now also U71.8 (A6); no longer U71.3 (A1)
- net B10: now also U70.7 (A5); no longer U70.4 (A2)
- net B11: now also U70.6 (A4); no longer U70.5 (A3)
- net B12: now also U70.5 (A3); no longer U70.6 (A4)
- net B13: now also U70.4 (A2); no longer U70.7 (A5)
- net B14: now also U70.3 (A1); no longer U70.8 (A6)
- net B15: now also U70.2 (A0); no longer U70.9 (A7)
- net B2: now also U71.7 (A5); no longer U71.4 (A2)
- net B3: now also U71.6 (A4); no longer U71.5 (A3)
- net B4: now also U71.5 (A3); no longer U71.6 (A4)
- net B5: now also U71.4 (A2); no longer U71.7 (A5)
- net B6: now also U71.3 (A1); no longer U71.8 (A6)
- net B7: now also U71.2 (A0); no longer U71.9 (A7)
- net B8: now also U70.9 (A7); no longer U70.2 (A0)
- net B9: now also U70.8 (A6); no longer U70.3 (A1)
Changed lines of the file:
@@
 $Descr A4 11693 8268
 encoding utf-8
-Sheet 14 18
+Sheet 13 18
 Title ""
 Date ""
@@
 Text Notes 5550 1800 0    50   ~ 10
 16-Bit Common Bus
+Text HLabel 7600 5050 3    50   BiDi ~ 0
+ARDUINO_IO_1
+Text HLabel 7700 5050 3    50   BiDi ~ 0
+ARDUINO_IO_2
+Text HLabel 7500 5050 3    50   BiDi ~ 0
+ARDUINO_IO_0
+Text HLabel 7800 5050 3    50   BiDi ~ 0
+ARDUINO_IO_3
+Text HLabel 8000 5050 3    50   BiDi ~ 0
+ARDUINO_IO_5
+Text HLabel 8100 5050 3    50   BiDi ~ 0
+ARDUINO_IO_6
+Text HLabel 8200 5050 3    50   BiDi ~ 0
+ARDUINO_IO_7
+Text HLabel 5500 5050 3    50   BiDi ~ 0
+ARDUINO_IO_8
 Text HLabel 5600 5050 3    50   BiDi ~ 0
-ARDUINO_IO_1
+ARDUINO_IO_9
 Text HLabel 5700 5050 3    50   BiDi ~ 0
-ARDUINO_IO_2
-Text HLabel 5500 5050 3    50   BiDi ~ 0
-ARDUINO_IO_0
+ARDUINO_IO_10
 Text HLabel 5800 5050 3    50   BiDi ~ 0
-ARDUINO_IO_3
+ARDUINO_IO_11
+Text HLabel 5900 5050 3    50   BiDi ~ 0
+ARDUINO_IO_12
 Text HLabel 6000 5050 3    50   BiDi ~ 0
-ARDUINO_IO_5
+ARDUINO_IO_13
 Text HLabel 6100 5050 3    50   BiDi ~ 0
-ARDUINO_IO_6
+ARDUINO_IO_14
 Text HLabel 6200 5050 3    50   BiDi ~ 0
-ARDUINO_IO_7
-Text HLabel 7500 5050 3    50   BiDi ~ 0
-ARDUINO_IO_8
-Text HLabel 7600 5050 3    50   BiDi ~ 0
-ARDUINO_IO_9
-Text HLabel 7700 5050 3    50   BiDi ~ 0
-ARDUINO_IO_10
-Text HLabel 7800 5050 3    50   BiDi ~ 0
-ARDUINO_IO_11
+ARDUINO_IO_15
 Text HLabel 7900 5050 3    50   BiDi ~ 0
-ARDUINO_IO_12
-Text HLabel 8000 5050 3    50   BiDi ~ 0
-ARDUINO_IO_13
-Text HLabel 8100 5050 3    50   BiDi ~ 0
-ARDUINO_IO_14
-Text HLabel 8200 5050 3    50   BiDi ~ 0
-ARDUINO_IO_15
-Text HLabel 5900 5050 3    50   BiDi ~ 0
 ARDUINO_IO_4
 Text HLabel 4300 5000 3    50   Output ~ 0
@@
 Text HLabel 4150 5000 3    50   Output ~ 0
 R-~W~_ARDUINO
-Text Label 8200 1950 3    50   ~ 0
+Text Label 7500 2050 3    50   ~ 0
 B0
-Text Label 8100 1950 3    50   ~ 0
+Text Label 7600 2050 3    50   ~ 0
 B1
-Text Label 8000 1950 3    50   ~ 0
+Text Label 7700 2050 3    50   ~ 0
 B2
-Text Label 7900 1950 3    50   ~ 0
+Text Label 7800 2050 3    50   ~ 0
 B3
-Text Label 7800 1950 3    50   ~ 0
+Text Label 7900 2050 3    50   ~ 0
 B4
-Text Label 7700 1950 3    50   ~ 0
+Text Label 8000 2050 3    50   ~ 0
 B5
-Text Label 7600 1950 3    50   ~ 0
+Text Label 8100 2050 3    50   ~ 0
 B6
-Text Label 7500 1950 3    50   ~ 0
+Text Label 8200 2050 3    50   ~ 0
 B7
-Text Label 6200 1950 3    50   ~ 0
+Text Label 5500 2050 3    50   ~ 0
 B8
-Text Label 6100 1950 3    50   ~ 0
+Text Label 5600 2050 3    50   ~ 0
 B9
-Text Label 6000 2050 1    50   ~ 0
+Text Label 5700 2150 1    50   ~ 0
 B10
-Text Label 5900 2050 1    50   ~ 0
+Text Label 5800 2150 1    50   ~ 0
 B11
-Text Label 5800 2050 1    50   ~ 0
+Text Label 5900 2150 1    50   ~ 0
 B12
-Text Label 5700 2050 1    50   ~ 0
+Text Label 6000 2150 1    50   ~ 0
 B13
-Text Label 5600 2050 1    50   ~ 0
+Text Label 6100 2150 1    50   ~ 0
 B14
-Text Label 5500 2050 1    50   ~ 0
+Text Label 6200 2150 1    50   ~ 0
 B15
 Text HLabel 3700 1800 0    50   BiDi ~ 0
