File: KiCad/breadboard_comp/Instr_Register.sch (KiCad schematic (older format))
At the start: 38 parts, among them U43 74LS08, U44 74LS273, U45 74LS273, U46 74LS245, U47 74LS245

Commit message: Computer built
Connections:
- net B0: now also U47.9 (A7); no longer U47.2 (A0)
- net B1: now also U47.8 (A6); no longer U47.3 (A1)
- net B10: now also U46.7 (A5); no longer U46.4 (A2)
- net B11: now also U46.6 (A4); no longer U46.5 (A3)
- net B12: now also U46.5 (A3); no longer U46.6 (A4)
- net B13: now also U46.4 (A2); no longer U46.7 (A5)
- net B14: now also U46.3 (A1); no longer U46.8 (A6)
- net B15: now also U46.2 (A0); no longer U46.9 (A7)
- net B2: now also U47.7 (A5); no longer U47.4 (A2)
- net B3: now also U47.6 (A4); no longer U47.5 (A3)
- net B4: now also U47.5 (A3); no longer U47.6 (A4)
- net B5: now also U47.4 (A2); no longer U47.7 (A5)
- net B6: now also U47.3 (A1); no longer U47.8 (A6)
- net B7: now also U47.2 (A0); no longer U47.9 (A7)
- net B8: now also U46.9 (A7); no longer U46.2 (A0)
- net B9: now also U46.8 (A6); no longer U46.3 (A1)
- net GND: now also U46.17 (B1), U46.18 (B0); no longer U46.11 (B7), U46.12 (B6)
- net at D72.2 (A), U44.5 (Q1): now also U46.12 (B6); no longer U46.17 (B1)
- net at D73.2 (A), U44.2 (Q0): now also U46.11 (B7); no longer U46.18 (B0)
- net at D75.2 (A), U45.16 (Q6): now also U47.17 (B1); no longer U47.12 (B6)
- net at D77.2 (A), U45.12 (Q4): now also U47.15 (B3); no longer U47.14 (B4)
- net at D81.2 (A), U45.2 (Q0): now also U47.11 (B7); no longer U47.18 (B0)
- net at D74.2 (A), U45.19 (Q7): now also U47.18 (B0); no longer U47.11 (B7)
- net at D76.2 (A), U45.15 (Q5): now also U47.16 (B2); no longer U47.13 (B5)
- net at D78.2 (A), U45.9 (Q3): now also U47.14 (B4); no longer U47.15 (B3)
- net at D79.2 (A), U45.6 (Q2): now also U47.13 (B5); no longer U47.16 (B2)
- net at D80.2 (A), U45.5 (Q1): now also U47.12 (B6); no longer U47.17 (B1)
Changed lines of the file:
@@
 $Descr A4 11693 8268
 encoding utf-8
-Sheet 8 18
+Sheet 18 18
 Title ""
 Date ""
@@
 Wire Wire Line
 	9500 2500 9500 3250
-Text Label 9500 2600 1    50   ~ 0
+Text Label 8800 2600 1    50   ~ 0
 B0
-Text Label 9400 2650 1    50   ~ 0
+Text Label 8900 2650 1    50   ~ 0
 B1
-Text Label 9300 2750 1    50   ~ 0
+Text Label 9000 2750 1    50   ~ 0
 B2
-Text Label 9200 2800 1    50   ~ 0
+Text Label 9100 2800 1    50   ~ 0
 B3
-Text Label 9100 2850 1    50   ~ 0
+Text Label 9200 2850 1    50   ~ 0
 B4
-Text Label 9000 2900 1    50   ~ 0
+Text Label 9300 2900 1    50   ~ 0
 B5
-Text Label 8900 2950 1    50   ~ 0
+Text Label 9400 2950 1    50   ~ 0
 B6
-Text Label 8800 3000 1    50   ~ 0
+Text Label 9500 3000 1    50   ~ 0
 B7
 Entry Wire Line
@@
 Wire Wire Line
 	7350 2500 7350 3250
-Text Label 7350 2600 1    50   ~ 0
+Text Label 6650 2600 1    50   ~ 0
 B8
-Text Label 7250 2650 1    50   ~ 0
+Text Label 6750 2650 1    50   ~ 0
 B9
-Text Label 7150 2750 1    50   ~ 0
+Text Label 6850 2750 1    50   ~ 0
 B10
-Text Label 7050 2800 1    50   ~ 0
+Text Label 6950 2800 1    50   ~ 0
 B11
-Text Label 6950 2850 1    50   ~ 0
+Text Label 7050 2850 1    50   ~ 0
 B12
-Text Label 6850 2900 1    50   ~ 0
+Text Label 7150 2900 1    50   ~ 0
 B13
-Text Label 6750 2950 1    50   ~ 0
+Text Label 7250 2950 1    50   ~ 0
 B14
-Text Label 6650 3000 1    50   ~ 0
+Text Label 7350 3000 1    50   ~ 0
 B15
 Wire Wire Line
 	2650 4250 2650 4650
 Wire Wire Line
-	7350 4650 7350 4250
-Wire Wire Line
 	2550 4250 2550 4750
 Wire Wire Line
-	7250 4750 7250 4250
-Wire Wire Line
 	2450 4250 2450 4850
 Wire Wire Line
@@
 	5150 4250 5150 5650
 Wire Wire Line
-	9500 5650 9500 4250
-Wire Wire Line
 	5050 4250 5050 5750
 Wire Wire Line
-	9400 5750 9400 4250
-Wire Wire Line
 	4950 4250 4950 5850
 Wire Wire Line
 	4950 5850 5550 5850
 Wire Wire Line
-	9300 5850 9300 4250
-Wire Wire Line
 	4850 4250 4850 5950
 Wire Wire Line
-	9200 5950 9200 4250
-Wire Wire Line
 	4750 4250 4750 6050
 Wire Wire Line
-	9100 6050 9100 4250
-Wire Wire Line
 	4650 4250 4650 6150
 Wire Wire Line
-	9000 6150 9000 4250
-Wire Wire Line
 	4550 4250 4550 6250
 Wire Wire Line
-	8900 6250 8900 4250
-Wire Wire Line
 	4450 4250 4450 6350
 Wire Wire Line
 	4450 6350 4550 6350
-Wire Wire Line
-	8800 6350 8800 4250
 $Comp
 L power:GND #PWR?
@@
 Connection ~ 4350 4650
 Wire Wire Line
-	4350 4650 7350 4650
+	4350 4650 6650 4650
 Wire Wire Line
 	4150 4750 4150 6700
@@
 Connection ~ 4550 6350
 Wire Wire Line
-	4550 6350 8800 6350
-Wire Wire Line
 	4750 6700 4750 6250
 Wire Wire Line
@@
 Connection ~ 4750 6250
 Wire Wire Line
-	4750 6250 8900 6250
-Wire Wire Line
 	4950 6700 4950 6150
 Wire Wire Line
@@
 Connection ~ 4950 6150
 Wire Wire Line
-	4950 6150 9000 6150
-Wire Wire Line
 	5150 6700 5150 6050
 Wire Wire Line
@@
 Connection ~ 5150 6050
 Wire Wire Line
-	5150 6050 9100 6050
-Wire Wire Line
 	5350 6700 5350 5950
 Wire Wire Line
@@
 Connection ~ 5350 5950
 Wire Wire Line
-	5350 5950 9200 5950
+	5350 5950 9100 5950
 Wire Wire Line
 	5550 6700 5550 5850
 Connection ~ 5550 5850
 Wire Wire Line
-	5550 5850 9300 5850
+	5550 5850 9000 5850
 Wire Wire Line
 	5750 6700 5750 5750
@@
 Connection ~ 5750 5750
 Wire Wire Line
-	5750 5750 9400 5750
+	5750 5750 8900 5750
 Wire Wire Line
 	5950 6700 5950 5650
@@
 Connection ~ 5950 5650
 Wire Wire Line
-	5950 5650 9500 5650
+	5950 5650 8800 5650
 Wire Wire Line
 	1250 2150 6350 2150
@@
 Connection ~ 1750 1900
 Connection ~ 4150 4750
-Wire Wire Line
-	4150 4750 7250 4750
 $Comp
 L power:GND #PWR0100
 U 1 1 5EFB5A5B
-P 6900 4400
-F 0 "#PWR0100" H 6900 4150 50  0001 C CNN
-F 1 "GND" H 6905 4227 50  0000 C CNN
-F 2 "" H 6900 4400 50  0001 C CNN
-F 3 "" H 6900 4400 50  0001 C CNN
-	1    6900 4400
-	1    0    0    -1
-$EndComp
-Wire Wire Line
-	6650 4250 6650 4350
-Wire Wire Line
-	6650 4350 6750 4350
+P 7100 4400
+F 0 "#PWR0100" H 7100 4150 50  0001 C CNN
+F 1 "GND" H 7105 4227 50  0000 C CNN
+F 2 "" H 7100 4400 50  0001 C CNN
+F 3 "" H 7100 4400 50  0001 C CNN
+	1    7100 4400
+	1    0    0    -1
+$EndComp
+Wire Wire Line
+	6850 4250 6850 4350
+Wire Wire Line
+	6850 4350 6950 4350
+Wire Wire Line
+	7350 4350 7350 4250
+Wire Wire Line
+	7250 4250 7250 4350
+Connection ~ 7250 4350
+Wire Wire Line
+	7250 4350 7350 4350
+Wire Wire Line
+	7100 4350 7100 4400
+Connection ~ 7100 4350
+Wire Wire Line
+	7100 4350 7150 4350
 Wire Wire Line
 	7150 4350 7150 4250
+Connection ~ 7150 4350
+Wire Wire Line
+	7150 4350 7250 4350
 Wire Wire Line
 	7050 4250 7050 4350
 Connection ~ 7050 4350
 Wire Wire Line
-	7050 4350 7150 4350
-Wire Wire Line
-	6900 4350 6900 4400
-Connection ~ 6900 4350
-Wire Wire Line
-	6900 4350 6950 4350
+	7050 4350 7100 4350
 Wire Wire Line
 	6950 4350 6950 4250
@@
 Wire Wire Line
 	6950 4350 7050 4350
-Wire Wire Line
-	6850 4250 6850 4350
-Connection ~ 6850 4350
-Wire Wire Line
-	6850 4350 6900 4350
-Wire Wire Line
-	6750 4350 6750 4250
-Connection ~ 6750 4350
-Wire Wire Line
-	6750 4350 6850 4350
 Text HLabel 2200 5700 0    50   Output ~ 0
 IR10
@@
 Text HLabel 9600 2400 2    50   BiDi ~ 0
 BUS
+Wire Wire Line
+	4150 4750 6750 4750
+Wire Wire Line
+	8800 4250 8800 5650
+Wire Wire Line
+	8900 5750 8900 4250
+Wire Wire Line
+	9000 4250 9000 5850
+Wire Wire Line
+	9100 5950 9100 4250
+Wire Wire Line
+	5150 6050 9200 6050
+Wire Wire Line
+	9200 4250 9200 6050
+Wire Wire Line
+	9300 6150 9300 4250
+Wire Wire Line
+	4950 6150 9300 6150
+Wire Wire Line
+	9400 4250 9400 6250
+Wire Wire Line
+	4750 6250 9400 6250
+Wire Wire Line
+	9500 6350 9500 4250
+Wire Wire Line
+	4550 6350 9500 6350
+Wire Wire Line
+	6650 4250 6650 4650
+Wire Wire Line
+	6750 4750 6750 4250
 Wire Bus Line
 	1850 2400 9600 2400
