File: KiCad/breadboard_comp/Instr_Register.sch (KiCad schematic (older format))
At the start: 38 parts, among them U43 74LS08, U44 74LS273, U45 74LS273, U46 74LS245, U47 74LS245

Commit message: Schematic + Report Progress
Parts:
- added C32: 0.01uF, symbol Device:C
- added R198: 100, symbol Device:R
- added U58, U74: 74LS08, symbol 74xx:74LS08
Connections:
- net GND: now also C32.2
- net II: now also U74.4, U74.5; no longer U43.2
- new net: U43.2, U58.8
- new net: R198.1, U74.6
- new net: C32.1, R198.2, U58.10, U58.9
Changed lines of the file:
@@
 $Descr A4 11693 8268
 encoding utf-8
-Sheet 18 19
+Sheet 18 18
 Title ""
 Date ""
@@
 Text HLabel 750  1800 0    50   Input ~ 0
 CLK
-Text HLabel 750  2000 0    50   Input ~ 0
+Text HLabel 3250 1250 2    50   Input ~ 0
 II
 Text HLabel 1250 2150 0    50   Input ~ 0
@@
 	750  1800 1000 1800
 Wire Wire Line
-	1000 2000 750  2000
-Wire Wire Line
 	1600 1900 1750 1900
 Wire Wire Line
@@
 Wire Wire Line
 	6750 4750 6750 4250
+$Comp
+L Device:R R?
+U 1 1 5F68327F
+P 1950 1250
+AR Path="/5F50482F/5F68327F" Ref="R?"  Part="1"
+AR Path="/5F46F293/5F68327F" Ref="R?"  Part="1"
+AR Path="/5EF95BB7/5F68327F" Ref="R198"  Part="1"
+F 0 "R198" H 2020 1296 50  0000 L CNN
+F 1 "100" V 1950 1200 50  0000 L CNN
+F 2 "" V 1880 1250 50  0001 C CNN
+F 3 "~" H 1950 1250 50  0001 C CNN
+	1    1950 1250
+	0    1    1    0
+$EndComp
+$Comp
+L Device:C C?
+U 1 1 5F683285
+P 1700 1000
+AR Path="/5F50482F/5F683285" Ref="C?"  Part="1"
+AR Path="/5F46F293/5F683285" Ref="C?"  Part="1"
+AR Path="/5EF95BB7/5F683285" Ref="C32"  Part="1"
+F 0 "C32" V 1448 1000 50  0000 C CNN
+F 1 "0.01uF" V 1539 1000 50  0000 C CNN
+F 2 "" H 1738 850 50  0001 C CNN
+F 3 "~" H 1700 1000 50  0001 C CNN
+	1    1700 1000
+	-1   0    0    1
+$EndComp
+Wire Wire Line
+	1700 1250 1700 1150
+Connection ~ 1700 1250
+Wire Wire Line
+	1700 1250 1800 1250
+$Comp
+L power:GND #PWR?
+U 1 1 5F68328E
+P 1850 700
+AR Path="/5F50482F/5F68328E" Ref="#PWR?"  Part="1"
+AR Path="/5F46F293/5F68328E" Ref="#PWR?"  Part="1"
+AR Path="/5EF95BB7/5F68328E" Ref="#PWR0288"  Part="1"
+F 0 "#PWR0288" H 1850 450 50  0001 C CNN
+F 1 "GND" H 1855 527 50  0000 C CNN
+F 2 "" H 1850 700 50  0001 C CNN
+F 3 "" H 1850 700 50  0001 C CNN
+	1    1850 700
+	0    -1   -1   0
+$EndComp
+Wire Wire Line
+	1700 700  1700 850
+Wire Wire Line
+	1700 700  1850 700
+$Comp
+L 74xx:74LS08 U?
+U 2 1 5F683296
+P 2750 1250
+AR Path="/5F46F293/5F683296" Ref="U?"  Part="2"
+AR Path="/5EF95BB7/5F683296" Ref="U74"  Part="2"
+F 0 "U74" H 2750 1575 50  0000 C CNN
+F 1 "74LS08" H 2750 1484 50  0000 C CNN
+F 2 "" H 2750 1250 50  0001 C CNN
+F 3 "http://www.ti.com/lit/gpn/sn74LS08" H 2750 1250 50  0001 C CNN
+	2    2750 1250
+	-1   0    0    1
+$EndComp
+$Comp
+L 74xx:74LS08 U?
+U 3 1 5F68329C
+P 1200 1250
+AR Path="/5F46F293/5F68329C" Ref="U?"  Part="3"
+AR Path="/5EF95BB7/5F68329C" Ref="U58"  Part="3"
+F 0 "U58" H 1200 1575 50  0000 C CNN
+F 1 "74LS08" H 1200 1484 50  0000 C CNN
+F 2 "" H 1200 1250 50  0001 C CNN
+F 3 "http://www.ti.com/lit/gpn/sn74LS08" H 1200 1250 50  0001 C CNN
+	3    1200 1250
+	-1   0    0    1
+$EndComp
+Wire Wire Line
+	1700 1250 1600 1250
+Wire Wire Line
+	1600 1250 1600 1350
+Wire Wire Line
+	1600 1350 1500 1350
+Connection ~ 1600 1250
+Wire Wire Line
+	1500 1150 1600 1150
+Wire Wire Line
+	1600 1150 1600 1250
+Wire Wire Line
+	2450 1250 2100 1250
+Wire Wire Line
+	3250 1250 3150 1250
+Wire Wire Line
+	3150 1250 3150 1150
+Wire Wire Line
+	3150 1150 3050 1150
+Wire Wire Line
+	3050 1350 3150 1350
+Wire Wire Line
+	3150 1350 3150 1250
+Connection ~ 3150 1250
+Wire Wire Line
+	900  1250 500  1250
+Wire Wire Line
+	500  1250 500  2000
+Wire Wire Line
+	500  2000 1000 2000
 Wire Bus Line
 	1850 2400 9600 2400
