File: KiCad/breadboard_comp/Program_Counter.sch (KiCad schematic (older format))
At the start: 8 parts, among them U57 74LS04, U58 74LS08, U59 74LS161, U60 74LS245, U61 74LS161, U62 74LS245, U63 74LS161

Commit message: Order Lists
Connections:
- net at U58.3, U63.1 (~MR): now also U59.1 (~MR), U61.1 (~MR)
Changed lines of the file:
@@
 	2600 1500 2600 1600
-Wire Wire Line
-	2600 1600 6950 1600
 Wire Wire Line
 	6950 1600 6950 2700
@@
 	1    0    0    -1
 $EndComp
+Text HLabel 3150 1050 0    50   BiDi ~ 0
+BUS
+Text HLabel 3450 6500 0    50   BiDi ~ 0
+BUS
+Wire Wire Line
+	4850 2700 4850 1600
+Connection ~ 4850 1600
+Wire Wire Line
+	4850 1600 6950 1600
+Wire Wire Line
+	2750 2700 2750 1600
+Wire Wire Line
+	2600 1600 2750 1600
 Wire Bus Line
 	3150 1050 7900 1050
 Wire Bus Line
 	3450 6500 7350 6500
-Text HLabel 3150 1050 0    50   BiDi ~ 0
-BUS
-Text HLabel 3450 6500 0    50   BiDi ~ 0
-BUS
+Connection ~ 2750 1600
+Wire Wire Line
+	2750 1600 4850 1600
 $EndSCHEMATC

Commit message: Computer built
Connections:
- net B0: now also U62.9 (A7); no longer U62.18 (B0)
- net B1: now also U62.8 (A6); no longer U62.17 (B1)
- net B2: now also U62.7 (A5); no longer U62.16 (B2)
- net B3: now also U62.6 (A4); no longer U62.15 (B3)
- net B4: now also U62.5 (A3); no longer U62.14 (B4)
- net B5: now also U62.4 (A2); no longer U62.13 (B5)
- net B6: now also U62.3 (A1); no longer U62.12 (B6)
- net B7: now also U62.2 (A0); no longer U62.11 (B7)
- net B8: now also U60.9 (A7); no longer U60.18 (B0)
- net B9: now also U60.8 (A6); no longer U60.17 (B1)
- net CE: no longer U59.10 (CET), U61.10 (CET)
- net CLK: now also U59.2 (CP), U61.2 (CP)
- net GND: now also U60.1 (A->B), U60.13 (B5), U60.14 (B4), U60.15 (B3), U60.16 (B2), U60.17 (B1), U60.18 (B0), U62.1 (A->B); no longer U60.4 (A2), U60.5 (A3), U60.6 (A4), U60.7 (A5), U60.8 (A6), U60.9 (A7)
- net VCC: no longer U60.1 (A->B), U62.1 (A->B)
- net at U63.11 (Q3): now also U62.14 (B4); no longer U62.5 (A3)
- net at U63.12 (Q2): now also U62.13 (B5); no longer U62.4 (A2)
- net at U63.13 (Q1): now also U62.12 (B6); no longer U62.3 (A1)
- net at U63.14 (Q0): now also U62.11 (B7); no longer U62.2 (A0)
- net at U63.15 (TC): now also U61.10 (CET); no longer U61.2 (CP)
- net at U61.11 (Q3): now also U62.18 (B0); no longer U62.9 (A7)
- net at U61.12 (Q2): now also U62.17 (B1); no longer U62.8 (A6)
- net at U61.13 (Q1): now also U62.16 (B2); no longer U62.7 (A5)
- net at U61.14 (Q0): now also U62.15 (B3); no longer U62.6 (A4)
- net at U61.15 (TC): now also U59.10 (CET); no longer U59.2 (CP)
- net at U59.13 (Q1): now also U60.12 (B6); no longer U60.3 (A1)
- net at U59.14 (Q0): now also U60.11 (B7); no longer U60.2 (A0)
- new net B10: U60.7 (A5)
- new net B11: U60.6 (A4)
- new net B12: U60.5 (A3)
- new net B13: U60.4 (A2)
- new net B14: U60.3 (A1)
- new net B15: U60.2 (A0)
- no-connect marks 8 -> 2
Other:
- moved on the sheet: C15, U60, U62
