File: KiCad/breadboard_comp/ShiftRegister.sch (KiCad schematic (older format))
At the start: 9 parts, among them U31 74LS194, U32 74LS194, U33 74LS245, U34 74LS194, U35 74LS245, U36 74LS194, U37 74LS32, U4 74LS32

Commit message: Computer built
Connections:
- net B0: now also U35.9 (A7); no longer U35.18 (B0)
- net B1: now also U35.8 (A6); no longer U35.17 (B1)
- net B10: now also U33.7 (A5); no longer U33.16 (B2)
- net B11: now also U33.6 (A4); no longer U33.15 (B3)
- net B12: now also U33.5 (A3); no longer U33.14 (B4)
- net B13: now also U33.4 (A2); no longer U33.13 (B5)
- net B14: now also U33.3 (A1); no longer U33.12 (B6)
- net B15: now also U33.2 (A0); no longer U33.11 (B7)
- net B2: now also U35.7 (A5); no longer U35.16 (B2)
- net B3: now also U35.6 (A4); no longer U35.15 (B3)
- net B4: now also U35.5 (A3); no longer U35.14 (B4)
- net B5: now also U35.4 (A2); no longer U35.13 (B5)
- net B6: now also U35.3 (A1); no longer U35.12 (B6)
- net B7: now also U35.2 (A0); no longer U35.11 (B7)
- net B8: now also U33.9 (A7); no longer U33.18 (B0)
- net B9: now also U33.8 (A6); no longer U33.17 (B1)
- net GND: now also U31.7 (Dsl), U33.1 (A->B), U35.1 (A->B), U36.2 (Dsr); no longer U31.2 (Dsr), U36.7 (Dsl)
- net VCC: no longer U33.1 (A->B), U35.1 (A->B)
- net at U31.12 (Q3): now also U33.18 (B0); no longer U33.9 (A7)
- net at U31.13 (Q2): now also U33.17 (B1); no longer U33.8 (A6)
- net at U31.14 (Q1): now also U33.16 (B2); no longer U33.7 (A5)
- net at U32.13 (Q2): now also U33.13 (B5); no longer U33.4 (A2)
- net at U32.14 (Q1): now also U33.12 (B6); no longer U33.3 (A1)
- net at U34.13 (Q2): now also U35.17 (B1); no longer U35.8 (A6)
- net at U34.14 (Q1): now also U35.16 (B2); no longer U35.7 (A5)
- net at U36.13 (Q2): now also U35.13 (B5); no longer U35.4 (A2)
- net at U36.14 (Q1): now also U35.12 (B6); no longer U35.3 (A1)
- net at U36.15 (Q0): now also U35.11 (B7); no longer U35.2 (A0)
- new net: U31.15 (Q0), U32.7 (Dsl), U33.15 (B3)
- new net: U31.2 (Dsr), U32.12 (Q3), U33.14 (B4)
- new net: U32.15 (Q0), U33.11 (B7), U34.7 (Dsl)
- new net: U32.2 (Dsr), U34.12 (Q3), U35.18 (B0)
- new net: U34.15 (Q0), U35.15 (B3), U36.7 (Dsl)
- new net: U34.2 (Dsr), U35.14 (B4), U36.12 (Q3)
