File: KiCad/breadboard_comp/breadboard_comp.sch (KiCad schematic (older format))
At the start: 48 parts

Commit message: Computer built
Changed lines of the file:
@@
-$EndSheet
-$Sheet
-S 2500 17000 1500 1000
-U 5EF95BB7
-F0 "Instruction Register" 50
-F1 "Instr_Register.sch" 50
-F2 "CLK" I R 4000 17100 50
-F3 "II" I R 4000 17400 50
-F4 "~RST" I R 4000 17200 50
-F5 "IR10" O L 2500 17900 50
-F6 "~IO" I R 4000 17300 50
-F7 "IR11" O L 2500 17800 50
-F8 "IR12" O L 2500 17700 50
-F9 "IR13" O L 2500 17600 50
-F10 "IR14" O L 2500 17500 50
-F11 "IR15" O L 2500 17400 50
-F12 "BUS" B R 4000 17700 50
 $EndSheet
 $Sheet
@@
 F39 "~ST_I" O R 4000 21750 50
 F40 "RI" O R 4000 21850 50
-F41 "~RO" O R 4000 21950 50
+F41 "RO" O R 4000 21950 50
 F42 "FI" O R 4000 22050 50
 $EndSheet
@@
 F10 "A8" I R 4000 11200 50
 F11 "A9" I R 4000 11300 50
-F12 "~RI" I R 4000 10100 50
-F13 "~RO" I R 4000 10000 50
+F12 "RI" I R 4000 10100 50
+F13 "RO" I R 4000 10000 50
 F14 "MEM_0" I R 4000 8100 50
 F15 "MEM_1" I R 4000 8200 50
@@
 Wire Bus Line
 	7650 3250 7650 7300
+$Sheet
+S 2500 17000 1500 1000
+U 5EF95BB7
+F0 "Instruction Register" 50
+F1 "Instr_Register.sch" 50
+F2 "CLK" I R 4000 17100 50
+F3 "II" I R 4000 17400 50
+F4 "~RST" I R 4000 17200 50
+F5 "IR10" O L 2500 17900 50
+F6 "~IO" I R 4000 17300 50
+F7 "IR11" O L 2500 17800 50
+F8 "IR12" O L 2500 17700 50
+F9 "IR13" O L 2500 17600 50
+F10 "IR14" O L 2500 17500 50
+F11 "IR15" O L 2500 17400 50
+F12 "BUS" B R 4000 17700 50
+$EndSheet
 Wire Bus Line
 	7650 19500 15550 19500
