File: KiCad/breadboard_comp/breadboard_comp.sch (KiCad schematic (older format))
At the start: 48 parts

Commit message: Schematic + Report Progress
Changed lines of the file:
@@
 $Descr A2 16535 23386 portrait
 encoding utf-8
-Sheet 1 19
+Sheet 1 18
 Title ""
 Date ""
@@
 F0 "Clock" 50
 F1 "clock.sch" 50
-F2 "~CLK" O R 4000 1300 50
-F3 "CLK" O R 4000 1150 50
-F4 "HLT" I R 4000 1950 50
+F2 "HLT" I R 4000 1950 50
+F3 "CLK0" O R 4000 1150 50
+F4 "CLK1" O R 4000 1250 50
+F5 "CLK2" O R 4000 1350 50
+F6 "CLK3" O R 4000 1450 50
+F7 "CLK4" O R 4000 1550 50
+F8 "CLK5" O R 4000 1650 50
+F9 "CLK6" O R 4000 1750 50
+F10 "CLK7" O R 4000 1850 50
 $EndSheet
 $Sheet
@@
 F1 "Display.sch" 50
 F2 "OUT" I L 11500 18200 50
-F3 "CLK" I L 11500 18100 50
-F4 "BUS" B L 11500 18400 50
+F3 "BUS" B L 11500 18400 50
 $EndSheet
 $Sheet
@@
 F0 "Control Logic" 50
 F1 "Control.sch" 50
-F2 "~CLK" I R 4000 18550 50
-F3 "IR_10" I L 2500 18550 50
-F4 "IR_11" I L 2500 18650 50
-F5 "IR_12" I L 2500 18750 50
-F6 "IR_13" I L 2500 18850 50
-F7 "IR_14" I L 2500 18950 50
-F8 "IR_15" I L 2500 19050 50
-F9 "CF_O" I R 4000 18650 50
-F10 "ZF_O" I R 4000 18750 50
-F11 "PF_O" I R 4000 18850 50
-F12 "CE" O R 4000 19050 50
-F13 "~RST" O R 4000 19150 50
-F14 "~CNT_O" O R 4000 19250 50
-F15 "MI" O R 4000 19350 50
-F16 "II" O R 4000 19450 50
-F17 "~IO" O R 4000 19550 50
-F18 "AI" O R 4000 19650 50
-F19 "BI" O R 4000 19750 50
-F20 "~BO" O R 4000 19850 50
-F21 "CI" O R 4000 19950 50
-F22 "~CO" O R 4000 20050 50
-F23 "SU" O R 4000 20150 50
-F24 "~EO" O R 4000 20250 50
-F25 "~SO" O R 4000 20350 50
-F26 "SI" O R 4000 20450 50
-F27 "SFL" O R 4000 20550 50
-F28 "SFR" O R 4000 20650 50
-F29 "~E" O R 4000 20750 50
-F30 "R_~W" O R 4000 20850 50
-F31 "OUT" O R 4000 20950 50
-F32 "DONE" O R 4000 21050 50
-F33 "~JMP" O R 4000 21150 50
-F34 "HLT" O R 4000 21250 50
-F35 "~AO" O R 4000 21350 50
-F36 "~ST_J" O R 4000 21450 50
-F37 "~ST_D" O R 4000 21550 50
-F38 "~ST_O" O R 4000 21650 50
-F39 "~ST_I" O R 4000 21750 50
-F40 "RI" O R 4000 21850 50
-F41 "RO" O R 4000 21950 50
-F42 "FI" O R 4000 22050 50
+F2 "IR_10" I L 2500 18550 50
+F3 "IR_11" I L 2500 18650 50
+F4 "IR_12" I L 2500 18750 50
+F5 "IR_13" I L 2500 18850 50
+F6 "IR_14" I L 2500 18950 50
+F7 "IR_15" I L 2500 19050 50
+F8 "CF_O" I R 4000 18650 50
+F9 "ZF_O" I R 4000 18750 50
+F10 "PF_O" I R 4000 18850 50
+F11 "CE" O R 4000 19050 50
+F12 "~RST" O R 4000 19150 50
+F13 "~CNT_O" O R 4000 19250 50
+F14 "MI" O R 4000 19350 50
+F15 "II" O R 4000 19450 50
+F16 "~IO" O R 4000 19550 50
+F17 "AI" O R 4000 19650 50
+F18 "BI" O R 4000 19750 50
+F19 "~BO" O R 4000 19850 50
+F20 "CI" O R 4000 19950 50
+F21 "~CO" O R 4000 20050 50
+F22 "SU" O R 4000 20150 50
+F23 "~EO" O R 4000 20250 50
+F24 "~SO" O R 4000 20350 50
+F25 "SI" O R 4000 20450 50
+F26 "SFL" O R 4000 20550 50
+F27 "SFR" O R 4000 20650 50
+F28 "~E" O R 4000 20750 50
+F29 "R_~W" O R 4000 20850 50
+F30 "OUT" O R 4000 20950 50
+F31 "DONE" O R 4000 21050 50
+F32 "~JMP" O R 4000 21150 50
+F33 "HLT" O R 4000 21250 50
+F34 "~AO" O R 4000 21350 50
+F35 "~ST_J" O R 4000 21450 50
+F36 "~ST_D" O R 4000 21550 50
+F37 "~ST_O" O R 4000 21650 50
+F38 "~ST_I" O R 4000 21750 50
+F39 "RI" O R 4000 21850 50
+F40 "RO" O R 4000 21950 50
+F41 "FI" O R 4000 22050 50
+F42 "CLK" I R 4000 18550 50
 $EndSheet
 $Sheet
@@
 	2000 3400 2000 3500
 Wire Wire Line
-	4000 1300 6500 1300
-Wire Wire Line
-	6500 18550 4000 18550
-Wire Wire Line
-	6500 1300 6500 18550
-Wire Wire Line
 	11500 1650 11000 1650
 Wire Wire Line
@@
 	10800 18850 4000 18850
 Wire Wire Line
-	4000 1150 6600 1150
-Wire Wire Line
-	10500 1150 10500 2600
-Wire Wire Line
-	10500 18100 11500 18100
-Connection ~ 10500 1150
-Wire Wire Line
-	11500 16600 10500 16600
-Connection ~ 10500 16600
-Wire Wire Line
-	10500 16600 10500 18100
-Wire Wire Line
-	10500 15100 11500 15100
-Connection ~ 10500 15100
-Wire Wire Line
-	10500 15100 10500 16600
-Wire Wire Line
-	11500 13600 10500 13600
-Connection ~ 10500 13600
-Wire Wire Line
-	10500 13600 10500 15100
-Wire Wire Line
-	10500 12100 11500 12100
-Connection ~ 10500 12100
-Wire Wire Line
-	10500 12100 10500 13600
-Wire Wire Line
-	11500 9600 10500 9600
-Connection ~ 10500 9600
-Wire Wire Line
-	10500 9600 10500 12100
-Wire Wire Line
-	10500 2600 11500 2600
-Connection ~ 10500 2600
-Wire Wire Line
-	10500 2600 10500 9600
-Wire Wire Line
-	11500 1150 10500 1150
-Wire Wire Line
-	6600 1150 6600 2600
-Wire Wire Line
-	6600 17100 4000 17100
-Connection ~ 6600 1150
-Wire Wire Line
-	6600 1150 10500 1150
-Wire Wire Line
-	4000 15100 6600 15100
-Connection ~ 6600 15100
-Wire Wire Line
-	6600 15100 6600 17100
-Wire Wire Line
-	4000 9900 6600 9900
-Connection ~ 6600 9900
-Wire Wire Line
-	6600 9900 6600 15100
-Wire Wire Line
-	4000 2600 6600 2600
-Connection ~ 6600 2600
-Wire Wire Line
-	6600 2600 6600 9900
-Wire Wire Line
 	4000 20950 10400 20950
 Wire Wire Line
 	10400 20950 10400 18200
-Wire Wire Line
-	10400 18200 11500 18200
 Wire Wire Line
 	4000 19150 6700 19150
@@
 F12 "BUS" B R 4000 17700 50
 $EndSheet
+Wire Wire Line
+	4000 18550 6550 18550
+Wire Wire Line
+	6550 18550 6550 1150
+Wire Wire Line
+	4000 1150 6550 1150
+Wire Wire Line
+	4000 1450 6450 1450
+Wire Wire Line
+	6450 1450 6450 17100
+Wire Wire Line
+	6450 17100 4000 17100
+Wire Wire Line
+	4000 15100 6350 15100
+Wire Wire Line
+	6350 15100 6350 1350
+Wire Wire Line
+	6350 1350 4000 1350
+Wire Wire Line
+	4000 1250 6250 1250
+Wire Wire Line
+	6250 1250 6250 9900
+Wire Wire Line
+	6250 9900 4000 9900
+Wire Wire Line
+	10400 1750 4000 1750
+Wire Wire Line
+	4000 1850 10500 1850
+Wire Wire Line
+	10400 18200 11500 18200
+Wire Wire Line
+	4000 1650 10600 1650
+Wire Wire Line
+	10600 15100 11500 15100
+Wire Wire Line
+	10600 1650 10600 12100
+Wire Wire Line
+	10400 1750 10400 16600
+Wire Wire Line
+	10400 16600 11500 16600
+Wire Wire Line
+	10500 1850 10500 2600
+Wire Wire Line
+	10500 2600 11500 2600
+Wire Wire Line
+	10700 1550 10700 9600
+Wire Wire Line
+	10700 9600 11500 9600
+Wire Wire Line
+	10250 1550 10250 1150
+Wire Wire Line
+	10250 1150 11500 1150
+Wire Wire Line
+	4000 1550 10250 1550
+Connection ~ 10250 1550
+Wire Wire Line
+	10250 1550 10700 1550
+Wire Wire Line
+	11500 12100 10600 12100
+Connection ~ 10600 12100
+Wire Wire Line
+	10600 12100 10600 13600
+Wire Wire Line
+	10600 13600 11500 13600
+Connection ~ 10600 13600
+Wire Wire Line
+	10600 13600 10600 15100
+Wire Wire Line
+	4000 5600 6000 5600
+Wire Wire Line
+	6000 5600 6000 9600
+Wire Wire Line
+	6000 9600 4000 9600
 Wire Bus Line
 	7650 19500 15550 19500
-$Sheet
-S 14250 15100 1200 1300
-U 5E9E51CE
-F0 "Test" 50
-F1 "test.sch" 50
-$EndSheet
 $EndSCHEMATC
