File: KiCad/breadboard_comp/FlagsRegister.sch (KiCad schematic (older format))
At the start: 3 parts, among them U64 74LS08, U65 74LS273

Commit message: Schematic + Report Progress
Parts:
- added C29: 0.01uF, symbol Device:C
- added R195: 100, symbol Device:R
- added U56, U58: 74LS08, symbol 74xx:74LS08
Connections:
- net FI: now also U58.4, U58.5; no longer U64.2
- net GND: now also C29.2
- new net: U56.8, U64.2
- new net: R195.1, U58.6
- new net: C29.1, R195.2, U56.10, U56.9
Other:
- moved on the sheet: C16, U64A, U65
