File: KiCad/breadboard_comp/MAR.sch (KiCad schematic (older format))
At the start: 14 parts, among them SW4 SW_SPDT, SW5 SW_SPDT, U54 74LS273, U55 74LS273, U56 74LS08

Commit message: Schematic + Report Progress
Parts:
- added C28: 0.01uF, symbol Device:C
- added R194: 100, symbol Device:R
- added U38: 74LS08, symbol 74xx:74LS08
- added unit 2 of U56
Connections:
- net GND: now also C28.2
- net MI: now also U56.4, U56.5; no longer U56.2
- new net: U38.8, U56.2
- new net: R194.1, U56.6
- new net: C28.1, R194.2, U38.10, U38.9
Changed lines of the file:
@@
 $Descr A4 11693 8268
 encoding utf-8
-Sheet 9 19
+Sheet 9 18
 Title ""
 Date ""
@@
 Text HLabel 5200 1100 2    50   Input ~ 0
 ~RST
-Text HLabel 5500 1750 2    50   Input ~ 0
+Text HLabel 6100 5250 3    50   Input ~ 0
 MI
 Entry Wire Line
@@
 Wire Wire Line
 	5500 1950 5250 1950
-Wire Wire Line
-	5250 1750 5500 1750
 Wire Wire Line
 	4650 1850 3700 1850
@@
 Wire Wire Line
 	4600 2000 4600 850
+$Comp
+L Device:R R?
+U 1 1 5F6C4BB2
+P 6100 3850
+AR Path="/5F50482F/5F6C4BB2" Ref="R?"  Part="1"
+AR Path="/5F46F293/5F6C4BB2" Ref="R?"  Part="1"
+AR Path="/5E4488B6/5F6C4BB2" Ref="R194"  Part="1"
+F 0 "R194" H 6170 3896 50  0000 L CNN
+F 1 "100" V 6100 3800 50  0000 L CNN
+F 2 "" V 6030 3850 50  0001 C CNN
+F 3 "~" H 6100 3850 50  0001 C CNN
+	1    6100 3850
+	-1   0    0    1
+$EndComp
+$Comp
+L Device:C C?
+U 1 1 5F6C4BB8
+P 6350 3600
+AR Path="/5F50482F/5F6C4BB8" Ref="C?"  Part="1"
+AR Path="/5F46F293/5F6C4BB8" Ref="C?"  Part="1"
+AR Path="/5E4488B6/5F6C4BB8" Ref="C28"  Part="1"
+F 0 "C28" V 6098 3600 50  0000 C CNN
+F 1 "0.01uF" V 6189 3600 50  0000 C CNN
+F 2 "" H 6388 3450 50  0001 C CNN
+F 3 "~" H 6350 3600 50  0001 C CNN
+	1    6350 3600
+	0    -1   -1   0
+$EndComp
+Wire Wire Line
+	6100 3600 6200 3600
+Connection ~ 6100 3600
+Wire Wire Line
+	6100 3600 6100 3700
+$Comp
+L power:GND #PWR?
+U 1 1 5F6C4BC1
+P 6650 3750
+AR Path="/5F50482F/5F6C4BC1" Ref="#PWR?"  Part="1"
+AR Path="/5F46F293/5F6C4BC1" Ref="#PWR?"  Part="1"
+AR Path="/5E4488B6/5F6C4BC1" Ref="#PWR0284"  Part="1"
+F 0 "#PWR0284" H 6650 3500 50  0001 C CNN
+F 1 "GND" H 6655 3577 50  0000 C CNN
+F 2 "" H 6650 3750 50  0001 C CNN
+F 3 "" H 6650 3750 50  0001 C CNN
+	1    6650 3750
+	1    0    0    -1
+$EndComp
+Wire Wire Line
+	6650 3600 6500 3600
+Wire Wire Line
+	6650 3600 6650 3750
+$Comp
+L 74xx:74LS08 U?
+U 2 1 5F6C4BC9
+P 6100 4650
+AR Path="/5F46F293/5F6C4BC9" Ref="U?"  Part="2"
+AR Path="/5E4488B6/5F6C4BC9" Ref="U56"  Part="2"
+F 0 "U56" H 6100 4975 50  0000 C CNN
+F 1 "74LS08" H 6100 4884 50  0000 C CNN
+F 2 "" H 6100 4650 50  0001 C CNN
+F 3 "http://www.ti.com/lit/gpn/sn74LS08" H 6100 4650 50  0001 C CNN
+	2    6100 4650
+	0    -1   -1   0
+$EndComp
+$Comp
+L 74xx:74LS08 U?
+U 3 1 5F6C4BCF
+P 6100 3100
+AR Path="/5F46F293/5F6C4BCF" Ref="U?"  Part="3"
+AR Path="/5E4488B6/5F6C4BCF" Ref="U38"  Part="3"
+F 0 "U38" H 6100 3425 50  0000 C CNN
+F 1 "74LS08" H 6100 3334 50  0000 C CNN
+F 2 "" H 6100 3100 50  0001 C CNN
+F 3 "http://www.ti.com/lit/gpn/sn74LS08" H 6100 3100 50  0001 C CNN
+	3    6100 3100
+	0    -1   -1   0
+$EndComp
+Wire Wire Line
+	6100 3600 6100 3500
+Wire Wire Line
+	6100 3500 6000 3500
+Wire Wire Line
+	6000 3500 6000 3400
+Connection ~ 6100 3500
+Wire Wire Line
+	6200 3400 6200 3500
+Wire Wire Line
+	6200 3500 6100 3500
+Wire Wire Line
+	6100 4350 6100 4000
+Wire Wire Line
+	6100 5250 6100 5100
+Wire Wire Line
+	6100 5100 6200 5100
+Wire Wire Line
+	6200 5100 6200 4950
+Wire Wire Line
+	6000 4950 6000 5100
+Wire Wire Line
+	6000 5100 6100 5100
+Connection ~ 6100 5100
+Wire Wire Line
+	6100 2800 6100 1750
+Wire Wire Line
+	5250 1750 6100 1750
 Wire Bus Line
 	500  750  5200 750
